Commit message: add wheel wheeled.py

File: resources/robots/four_wheeled/urdf/wheel_legged.urdf (robot description, URDF)
Before this commit: robot wheel_legged, 22 links, 21 joints
Links:
- link LF_calf: geometry collision box size=0.3 0.0258 0.02; visual mesh filename=../meshes/LF_calf.STL scale=1 1 1
- link LF_hip: geometry visual mesh filename=../meshes/LF_hip.STL scale=1 1 1
- link LF_thigh: geometry visual mesh filename=../meshes/LF_thigh.STL scale=1 1 1
- link LF_wheel: geometry collision cylinder length=0.001 radius=0.127; visual mesh filename=../meshes/LF_wheel.STL scale=1 1 1
- link LH_calf: geometry collision box size=0.3 0.0258 0.02; visual mesh filename=../meshes/LH_calf.STL scale=1 1 1
- link LH_hip: geometry visual mesh filename=../meshes/LH_hip.STL scale=1 1 1
- link LH_thigh: geometry visual mesh filename=../meshes/LH_thigh.STL scale=1 1 1
- link LH_wheel: geometry collision cylinder length=0.001 radius=0.127; visual mesh filename=../meshes/LH_wheel.STL scale=1 1 1
- link RF_calf: geometry collision box size=0.3 0.0258 0.02; visual mesh filename=../meshes/RF_calf.STL scale=1 1 1
- link RF_hip: geometry visual mesh filename=../meshes/RF_hip.STL scale=1 1 1
- link RF_thigh: geometry visual mesh filename=../meshes/RF_thigh.STL scale=1 1 1
- link RF_wheel: geometry collision cylinder length=0.001 radius=0.127; visual mesh filename=../meshes/RF_wheel.STL scale=1 1 1
- link RH_calf: geometry collision box size=0.3 0.0258 0.02; visual mesh filename=../meshes/RH_calf.STL scale=1 1 1
- link RH_hip: geometry visual mesh filename=../meshes/RH_hip.STL scale=1 1 1
- link RH_thigh: geometry visual mesh filename=../meshes/RH_thigh.STL scale=1 1 1
- link RH_wheel: geometry collision cylinder length=0.001 radius=0.127; visual mesh filename=../meshes/RH_wheel.STL scale=1 1 1
- link base: geometry collision box size=0.53 0.256 0.155; visual mesh filename=../meshes/base_link.STL scale=1 1 1
